File: pcb/ibc/ibc.kicad_sch (KiCad schematic)
At the start: 72 parts, among them J1 MOLEX_0039291067, J2 CONN_01X03, J3 CONN_01X05, J4 MOLEX_0532610571, J5 U.FL, J6 U.FL, J7 U.FL, J8 U.FL, J9 MOLEX_0039291087, M1 LOGO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

Commit message: Finished v0.1 IBC ready for fab
Parts:
- added J10, J11: GROUND, azonenberg_pcb:TESTPOINT_SMT_KEYSTONE_5016, symbol conn:CONN_01X01
Connections:
- net 12V0_OK: now also U1.12 (PA6); no longer U1.11 (PA5)
- net 12V0_OUT_EN: now also U1.10 (PA4); no longer U1.14 (PB0)
- net 12V0_REMOTE_VSENSE: now also U1.14 (PB0); no longer U1.15 (PB1)
- net 12V0_VSENSE: now also U1.15 (PB1); no longer U1.10 (PA4)
- net 12V_SHUNT_VOUT: now also U1.13 (PA7); no longer U1.7 (PA1)
- net 48V0_VSENSE: now also U1.8 (PA2); no longer U1.9 (PA3)
- net 48V_SHUNT_VOUT: now also U1.7 (PA1); no longer U1.8 (PA2)
- net GND: now also J10.1 (P1), J11.1 (P1)
- net LOAD_PGOOD: now also U1.9 (PA3); no longer U1.13 (PA7)
- net TEMP_ALERT: now also U1.11 (PA5); no longer U1.6 (PA0)
- no-connect marks 15 -> 16
Changed lines of the file:
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@@
   (title_block
     (title "48V -> 12V Intermediate Bus Converter")
-    (date "2023-10-15")
+    (date "2023-10-17")
     (rev "0.1")
     (company "Antikernel Labs")
@@
   (no_connect (at 359.41 81.28))
   (no_connect (at 33.02 104.14))
+  (no_connect (at 38.1 223.52))
   (no_connect (at 83.82 252.73))
   (no_connect (at 359.41 63.5))
@@
     (effects (font (size 1.27 1.27)) (justify left bottom))
   )
-  (label "12V0_REMOTE_VSENSE" (at 83.82 245.11 180)
+  (label "12V0_REMOTE_VSENSE" (at 83.82 242.57 180)
     (effects (font (size 1.27 1.27)) (justify right bottom))
   )
@@
     (effects (font (size 1.27 1.27)) (justify right bottom))
   )
-  (label "12V_SHUNT_VOUT" (at 38.1 226.06 180)
+  (label "12V_SHUNT_VOUT" (at 38.1 241.3 180)
     (effects (font (size 1.27 1.27)) (justify right bottom))
   )
@@
     (effects (font (size 1.27 1.27)) (justify left bottom))
   )
-  (label "48V_SHUNT_VOUT" (at 38.1 228.6 180)
+  (label "48V_SHUNT_VOUT" (at 38.1 226.06 180)
     (effects (font (size 1.27 1.27)) (justify right bottom))
   )
@@
     (effects (font (size 1.27 1.27)) (justify left bottom))
   )
+  (label "GND" (at 332.74 63.5 0)
+    (effects (font (size 1.27 1.27)) (justify left bottom))
+  )
   (label "12V0_SENSE" (at 133.35 132.08 0)
     (effects (font (size 1.27 1.27)) (justify left bottom))
@@
     (effects (font (size 1.27 1.27)) (justify left bottom))
   )
-  (label "12V0_OK" (at 38.1 236.22 180)
+  (label "12V0_OK" (at 38.1 238.76 180)
     (effects (font (size 1.27 1.27)) (justify right bottom))
   )
@@
     (effects (font (size 1.27 1.27)) (justify right bottom))
   )
-  (label "48V0_VSENSE" (at 38.1 231.14 180)
+  (label "48V0_VSENSE" (at 38.1 228.6 180)
     (effects (font (size 1.27 1.27)) (justify right bottom))
   )
@@
     (effects (font (size 1.27 1.27)) (justify right bottom))
   )
-  (label "LOAD_PGOOD" (at 38.1 241.3 180)
+  (label "LOAD_PGOOD" (at 38.1 231.14 180)
     (effects (font (size 1.27 1.27)) (justify right bottom))
   )
@@
     (effects (font (size 1.27 1.27)) (justify right bottom))
   )
+  (label "GND" (at 332.74 72.39 0)
+    (effects (font (size 1.27 1.27)) (justify left bottom))
+  )
   (label "12V_SHUNT_P" (at 33.02 121.92 180)
     (effects (font (size 1.27 1.27)) (justify right bottom))
@@
     (effects (font (size 1.27 1.27)) (justify left bottom))
   )
-  (label "12V0_OUT_EN" (at 83.82 242.57 180)
+  (label "12V0_OUT_EN" (at 38.1 233.68 180)
     (effects (font (size 1.27 1.27)) (justify right bottom))
   )
@@
     (effects (font (size 1.27 1.27)) (justify right bottom))
   )
-  (label "12V0_VSENSE" (at 38.1 233.68 180)
+  (label "12V0_VSENSE" (at 83.82 245.11 180)
     (effects (font (size 1.27 1.27)) (justify right bottom))
   )
@@
     (effects (font (size 1.27 1.27)) (justify right bottom))
   )
-  (label "TEMP_ALERT" (at 38.1 223.52 180)
+  (label "TEMP_ALERT" (at 38.1 236.22 180)
     (effects (font (size 1.27 1.27)) (justify right bottom))
   )
@@
       (effects (font (size 1.27 1.27)) hide)
     )
-    (pin "10" (alternate "ADC_IN4"))
+    (pin "10")
     (pin "11")
-    (pin "12" (alternate "ADC_IN6"))
-    (pin "13")
+    (pin "12")
+    (pin "13" (alternate "ADC_IN7"))
     (pin "18")
     (pin "19")
@@
     (pin "7" (alternate "ADC_IN1"))
     (pin "8" (alternate "ADC_IN2"))
-    (pin "9" (alternate "ADC_IN3"))
-    (pin "14")
+    (pin "9")
+    (pin "14" (alternate "ADC_IN8"))
     (pin "15" (alternate "ADC_IN9"))
     (pin "16")
@@
       (effects (font (size 1.27 1.27)) hide)
     )
-    (pin "10" (alternate "ADC_IN4"))
+    (pin "10")
     (pin "11")
-    (pin "12" (alternate "ADC_IN6"))
-    (pin "13")
+    (pin "12")
+    (pin "13" (alternate "ADC_IN7"))
     (pin "18")
     (pin "19")
@@
     (pin "7" (alternate "ADC_IN1"))
     (pin "8" (alternate "ADC_IN2"))
-    (pin "9" (alternate "ADC_IN3"))
-    (pin "14")
+    (pin "9")
+    (pin "14" (alternate "ADC_IN8"))
     (pin "15" (alternate "ADC_IN9"))
     (pin "16")
@@
       (effects (font (size 1.27 1.27)) hide)
     )
-    (pin "10" (alternate "ADC_IN4"))
+    (pin "10")
     (pin "11")
-    (pin "12" (alternate "ADC_IN6"))
-    (pin "13")
+    (pin "12")
+    (pin "13" (alternate "ADC_IN7"))
     (pin "18")
     (pin "19")
@@
     (pin "7" (alternate "ADC_IN1"))
     (pin "8" (alternate "ADC_IN2"))
-    (pin "9" (alternate "ADC_IN3"))
-    (pin "14")
+    (pin "9")
+    (pin "14" (alternate "ADC_IN8"))
     (pin "15" (alternate "ADC_IN9"))
     (pin "16")
@@
       (effects (font (size 1.27 1.27)) hide)
     )
-    (pin "10" (alternate "ADC_IN4"))
+    (pin "10")
     (pin "11")
-    (pin "12" (alternate "ADC_IN6"))
-    (pin "13")
+    (pin "12")
+    (pin "13" (alternate "ADC_IN7"))
     (pin "18")
     (pin "19")
@@
     (pin "7" (alternate "ADC_IN1"))
     (pin "8" (alternate "ADC_IN2"))
-    (pin "9" (alternate "ADC_IN3"))
-    (pin "14")
+    (pin "9")
+    (pin "14" (alternate "ADC_IN8"))
     (pin "15" (alternate "ADC_IN9"))
     (pin "16")
@@
     (pin "2")
   )
+  (symbol (lib_id "conn:CONN_01X01") (at 327.66 63.5 0) (mirror y) (unit 1)
+    (in_bom yes) (on_board yes) (fields_autoplaced)
+    (property "Reference" "J10" (id 0) (at 327.66 58.6572 0))
+    (property "Value" "GROUND" (id 1) (at 327.66 61.1941 0))
+    (property "Footprint" "azonenberg_pcb:TESTPOINT_SMT_KEYSTONE_5016" (id 2) (at 327.66 63.5 0)
+      (effects (font (size 1.27 1.27)) hide)
+    )
+    (property "Datasheet" "" (id 3) (at 327.66 63.5 0)
+      (effects (font (size 1.27 1.27)) hide)
+    )
+    (pin "1")
+  )
   (symbol (lib_id "analog-azonenberg:AD8218") (at 35.56 90.17 0) (unit 1)
     (in_bom yes) (on_board yes) (fields_autoplaced)
@@
     (pin "8")
   )
+  (symbol (lib_id "conn:CONN_01X01") (at 327.66 72.39 0) (mirror y) (unit 1)
+    (in_bom yes) (on_board yes) (fields_autoplaced)
+    (property "Reference" "J11" (id 0) (at 327.66 67.5472 0))
+    (property "Value" "GROUND" (id 1) (at 327.66 70.0841 0))
+    (property "Footprint" "azonenberg_pcb:TESTPOINT_SMT_KEYSTONE_5016" (id 2) (at 327.66 72.39 0)
+      (effects (font (size 1.27 1.27)) hide)
+    )
+    (property "Datasheet" "" (id 3) (at 327.66 72.39 0)
+      (effects (font (size 1.27 1.27)) hide)
+    )
+    (pin "1")
+  )
   (symbol (lib_id "device:R") (at 34.29 185.42 180) (unit 1)
     (in_bom yes) (on_board yes) (fields_autoplaced)
@@
       (reference "J9") (unit 1) (value "MOLEX_0039291087") (footprint "azonenberg_pcb:CONN_MOLEX_MINIFITJR_8POS_0039291087")
     )
+    (path "/9f938dc9-ea37-4d07-adbe-457c6fc2433f"
+      (reference "J10") (unit 1) (value "GROUND") (footprint "azonenberg_pcb:TESTPOINT_SMT_KEYSTONE_5016")
+    )
+    (path "/eb8d84f3-46e9-4cc9-932b-f019611c7325"
+      (reference "J11") (unit 1) (value "GROUND") (footprint "azonenberg_pcb:TESTPOINT_SMT_KEYSTONE_5016")
+    )
     (path "/00d6706d-789c-4d1c-89bd-f4ac91bb6505"

Commit message: Updated IBC board for v0.2 with antialiasing filter, plane fix, and 5V standby rail
Parts:
- added C18, C19: 0.47 uF, azonenberg_pcb:EIA_0402_CAP_NOSILK, symbol device:C
- added C20, C21: 2.2 uF, azonenberg_pcb:EIA_0805_CAP_NOSILK, symbol device:C
- added C22, C23: 4.7 uF, azonenberg_pcb:EIA_0603_CAP_NOSILK, symbol device:C
- added J12: U.FL, azonenberg_pcb:CONN_U.FL_TE_1909763-1, symbol conn:CONN_COAXIAL
- added L1, L2: 62 nH, azonenberg_pcb:EIA_0402_CAP_NOSILK, symbol device:L
- added R24: 10K, azonenberg_pcb:EIA_0402_RES_NOSILK, symbol device:R
- added TP2: TESTPOINT, azonenberg_pcb:TESTPOINT_SMT_0.5MM, symbol conn:CONN_01X01
- added U8: TPS7A2550DRVR, azonenberg_pcb:DFN_6_0.65MM_2x2MM, symbol power-azonenberg:TPS7A25
Connections:
- net 12V0_SWIN: now also C20.1, U8.4 (EN), U8.6 (IN)
- net 12V_SHUNT_VOUT: now also L2.2; no longer U1.13 (PA7)
- net 48V_SHUNT_VOUT: now also L1.2; no longer U1.7 (PA1)
- net GND: now also C18.2, C19.2, C20.2, C21.2, C22.1, C23.1, J12.2 (Ext), U8.5 (GND), U8.PAD (GND)
- net 5V0_SB: now reaches U3.2 (VS+)
- net 5V0_SB: now also U2.2 (VS+), C18.1, C19.1, C21.1, J12.1 (In), R24.2, U8.1 (OUT)
- new net 12V_SHUNT_FILT: C23.2, L2.1, U1.13 (PA7)
- new net 48V_SHUNT_FILT: C22.2, L1.1, U1.7 (PA1)
- new net 5V0_SB_PGOOD: R24.1, TP2.1 (P1), U8.3 (PG)
- no-connect marks 16 -> 14
Other:
- note added: "5V standby regulator Thermally limited to 142 mA"
- moved on the sheet: C7, R10, R11, U5

Commit message: Respun again for v0.3, moving 48V shunt outside high dI/dT loop because I was derpy
Connections:
- net 48V0: now also C1.1, C2.1
- net 48V_SHIN: no longer C1.1, C2.1
Other:
- moved on the sheet: C1, C2, R8
Changed lines of the file:
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@@
   (title_block
     (title "48V -> 12V Intermediate Bus Converter")
-    (date "2023-11-29")
-    (rev "0.2")
+    (date "2023-11-30")
+    (rev "0.3")
     (company "Antikernel Labs")
     (comment 1 "Andrew D. Zonenberg")
@@
   (junction (at 260.35 60.96) (diameter 0) (color 0 0 0 0)
   )
-  (junction (at 127 25.4) (diameter 0) (color 0 0 0 0)
-  )
   (junction (at 320.04 132.08) (diameter 0) (color 0 0 0 0)
   )
@@
   (junction (at 260.35 53.34) (diameter 0) (color 0 0 0 0)
   )
+  (junction (at 166.37 25.4) (diameter 0) (color 0 0 0 0)
+  )
   (junction (at 154.94 134.62) (diameter 0) (color 0 0 0 0)
   )
@@
   )
   (junction (at 33.02 114.3) (diameter 0) (color 0 0 0 0)
-  )
-  (junction (at 151.13 25.4) (diameter 0) (color 0 0 0 0)
   )
   (junction (at 287.655 25.4) (diameter 0) (color 0 0 0 0)
@@
     (stroke (width 0) (type default) (color 0 0 0 0))
   )
-  (wire (pts (xy 121.92 25.4) (xy 127 25.4))
+  (wire (pts (xy 121.92 25.4) (xy 134.62 25.4))
     (stroke (width 0) (type default) (color 0 0 0 0))
   )
@@
     (stroke (width 0) (type default) (color 0 0 0 0))
   )
-  (wire (pts (xy 151.13 25.4) (xy 175.26 25.4))
-    (stroke (width 0) (type default) (color 0 0 0 0))
-  )
   (wire (pts (xy 34.29 179.07) (xy 34.29 180.34))
     (stroke (width 0) (type default) (color 0 0 0 0))
@@
     (stroke (width 0) (type default) (color 0 0 0 0))
   )
-  (wire (pts (xy 127 33.02) (xy 151.13 33.02))
+  (wire (pts (xy 166.37 33.02) (xy 190.5 33.02))
     (stroke (width 0) (type default) (color 0 0 0 0))
   )
@@
     (stroke (width 0) (type default) (color 0 0 0 0))
   )
-  (wire (pts (xy 127 25.4) (xy 151.13 25.4))
+  (wire (pts (xy 166.37 25.4) (xy 190.5 25.4))
     (stroke (width 0) (type default) (color 0 0 0 0))
   )
@@
     (stroke (width 0) (type default) (color 0 0 0 0))
   )
-  (wire (pts (xy 190.5 25.4) (xy 198.12 25.4))
+  (wire (pts (xy 149.86 25.4) (xy 166.37 25.4))
     (stroke (width 0) (type default) (color 0 0 0 0))
   )
@@
     (effects (font (size 1.27 1.27)) (justify left bottom))
   )
-  (text "80.5 mW at 1.6A in" (at 175.26 34.29 0)
+  (text "80.5 mW at 1.6A in" (at 134.62 34.29 0)
     (effects (font (size 1.27 1.27)) (justify left bottom))
   )
@@
     (effects (font (size 1.27 1.27)) (justify right bottom))
   )
-  (label "48V0" (at 198.12 25.4 0)
+  (label "48V0" (at 157.48 25.4 0)
     (effects (font (size 1.27 1.27)) (justify left bottom))
   )
@@
     (effects (font (size 1.27 1.27)) (justify right bottom))
   )
-  (label "48V_SHUNT_N" (at 190.5 27.94 0)
+  (label "48V_SHUNT_N" (at 149.86 27.94 0)
     (effects (font (size 1.27 1.27)) (justify left bottom))
   )
@@
     (effects (font (size 1.27 1.27)) (justify right bottom))
   )
-  (label "48V_SHUNT_P" (at 175.26 27.94 180)
+  (label "48V_SHUNT_P" (at 134.62 27.94 180)
     (effects (font (size 1.27 1.27)) (justify right bottom))
   )
@@
     (effects (font (size 1.27 1.27)) (justify right bottom))
   )
-  (label "48V_SHIN" (at 175.26 25.4 180)
+  (label "48V_SHIN" (at 134.62 25.4 180)
     (effects (font (size 1.27 1.27)) (justify right bottom))
   )
@@
     (effects (font (size 1.27 1.27)) (justify left bottom))
   )
-  (label "GND" (at 151.13 33.02 0)
+  (label "GND" (at 190.5 33.02 0)
     (effects (font (size 1.27 1.27)) (justify left bottom))
   )
@@
     (pin "2")
   )
-  (symbol (lib_id "device:CP1") (at 151.13 29.21 0) (unit 1)
-    (in_bom yes) (on_board yes) (fields_autoplaced)
-    (property "Reference" "C2" (id 0) (at 154.051 27.7403 0)
-      (effects (font (size 1.27 1.27)) (justify left))
-    )
-    (property "Value" "PCR1J101MCL1GS" (id 1) (at 154.051 30.2772 0)
-      (effects (font (size 1.27 1.27)) (justify left))
-    )
-    (property "Footprint" "azonenberg_pcb:CAP_AL_10MM_SMT" (id 2) (at 151.13 29.21 0)
-      (effects (font (size 1.27 1.27)) hide)
-    )
-    (property "Datasheet" "" (id 3) (at 151.13 29.21 0)
+  (symbol (lib_id "device:CP1") (at 190.5 29.21 0) (unit 1)
+    (in_bom yes) (on_board yes) (fields_autoplaced)
+    (property "Reference" "C2" (id 0) (at 193.421 27.7403 0)
+      (effects (font (size 1.27 1.27)) (justify left))
+    )
+    (property "Value" "PCR1J101MCL1GS" (id 1) (at 193.421 30.2772 0)
+      (effects (font (size 1.27 1.27)) (justify left))
+    )
+    (property "Footprint" "azonenberg_pcb:CAP_AL_10MM_SMT" (id 2) (at 190.5 29.21 0)
+      (effects (font (size 1.27 1.27)) hide)
+    )
+    (property "Datasheet" "" (id 3) (at 190.5 29.21 0)
       (effects (font (size 1.27 1.27)) hide)
     )
@@
     (pin "2")
   )
-  (symbol (lib_id "device:CP1") (at 127 29.21 0) (unit 1)
-    (in_bom yes) (on_board yes) (fields_autoplaced)
-    (property "Reference" "C1" (id 0) (at 129.921 27.7403 0)
-      (effects (font (size 1.27 1.27)) (justify left))
-    )
-    (property "Value" "PCR1J101MCL1GS" (id 1) (at 129.921 30.2772 0)
-      (effects (font (size 1.27 1.27)) (justify left))
-    )
-    (property "Footprint" "azonenberg_pcb:CAP_AL_10MM_SMT" (id 2) (at 127 29.21 0)
-      (effects (font (size 1.27 1.27)) hide)
-    )
-    (property "Datasheet" "" (id 3) (at 127 29.21 0)
+  (symbol (lib_id "device:CP1") (at 166.37 29.21 0) (unit 1)
+    (in_bom yes) (on_board yes)
+    (property "Reference" "C1" (id 0) (at 170.18 27.9431 0)
+      (effects (font (size 1.27 1.27)) (justify left))
+    )
+    (property "Value" "PCR1J101MCL1GS" (id 1) (at 170.18 30.48 0)
+      (effects (font (size 1.27 1.27)) (justify left))
+    )
+    (property "Footprint" "azonenberg_pcb:CAP_AL_10MM_SMT" (id 2) (at 166.37 29.21 0)
+      (effects (font (size 1.27 1.27)) hide)
+    )
+    (property "Datasheet" "" (id 3) (at 166.37 29.21 0)
       (effects (font (size 1.27 1.27)) hide)
     )
@@
     (pin "PAD")
   )
-  (symbol (lib_id "passive-azonenberg:R-4TERM") (at 182.88 26.67 270) (mirror x) (unit 1)
+  (symbol (lib_id "passive-azonenberg:R-4TERM") (at 142.24 26.67 270) (mirror x) (unit 1)
     (in_bom yes) (on_board yes)
-    (property "Reference" "R8" (id 0) (at 182.88 21.8272 90))
-    (property "Value" "LVK24R025DER" (id 1) (at 182.88 30.48 90))
-    (property "Footprint" "azonenberg_pcb:OHMITE_LVK24" (id 2) (at 182.88 26.67 0)
+    (property "Reference" "R8" (id 0) (at 142.24 21.8272 90))
+    (property "Value" "LVK24R025DER" (id 1) (at 142.24 30.48 90))
+    (property "Footprint" "azonenberg_pcb:OHMITE_LVK24" (id 2) (at 142.24 26.67 0)
       (effects (font (size 1.524 1.524)) hide)
     )
-    (property "Datasheet" "" (id 3) (at 182.88 26.67 0)
+    (property "Datasheet" "" (id 3) (at 142.24 26.67 0)
       (effects (font (size 1.524 1.524)))
     )
