File: pcb/mainboard/fpgasupport.kicad_sch (KiCad schematic)
At the start: 30 parts, among them J5 XILINX_JTAG, M1 960-23-23-F-AB-0, U8 XC7K70T-2FBG484C

Commit message: Began assigning footprints
Parts:
- C113, C34, C35, C38, C39: footprint (none) -> azonenberg_pcb:EIA_1210_CAP_NOSILK
- C36, C40, C41: footprint (none) -> azonenberg_pcb:EIA_1206_CAP_NOSILK
- C42, C43, C44, C45, C46, C47, C48, C49, C50, C51, C52: footprint (none) -> azonenberg_pcb:EIA_0603_CAP_NOSILK
- J5: footprint (none) -> azonenberg_pcb:XILINX_JTAG_PTH_MOLEX_0878311420
- M1: footprint (none) -> azonenberg_pcb:HEATSINK_WAKEFIELDVETTE_960-23-23-F-AB-0
- R39, R40, R41, R42, R43, R44, R45, R46: footprint (none) -> azonenberg_pcb:EIA_0402_RES_NOSILK
- U8: footprint (none) -> azonenberg_pcb:BGA_484_22x22_FULLARRAY_1MM
Changed lines of the file:
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@@
       (effects (font (size 1.27 1.27)) (justify left))
     )
-    (property "Footprint" "" (id 2) (at 172.4152 205.74 0)
+    (property "Footprint" "azonenberg_pcb:EIA_0603_CAP_NOSILK" (id 2) (at 172.4152 205.74 0)
       (effects (font (size 1.27 1.27)) hide)
     )
@@
       (effects (font (size 1.524 1.524)) (justify left))
     )
-    (property "Footprint" "" (id 2) (at 35.56 60.96 0)
+    (property "Footprint" "azonenberg_pcb:XILINX_JTAG_PTH_MOLEX_0878311420" (id 2) (at 35.56 60.96 0)
       (effects (font (size 1.524 1.524)) hide)
     )
@@
     (property "Reference" "R45" (id 0) (at 68.58 162.56 90))
     (property "Value" "0" (id 1) (at 73.66 163.83 90))
-    (property "Footprint" "" (id 2) (at 73.66 165.608 90)
+    (property "Footprint" "azonenberg_pcb:EIA_0402_RES_NOSILK" (id 2) (at 73.66 165.608 90)
       (effects (font (size 1.27 1.27)) hide)
     )
@@
       (effects (font (size 1.27 1.27)) (justify left))
     )
-    (property "Footprint" "" (id 2) (at 79.7052 220.98 0)
+    (property "Footprint" "azonenberg_pcb:EIA_0603_CAP_NOSILK" (id 2) (at 79.7052 220.98 0)
       (effects (font (size 1.27 1.27)) hide)
     )
@@
       (effects (font (size 1.27 1.27)) (justify left))
     )
-    (property "Footprint" "" (id 2) (at 92.4052 220.98 0)
+    (property "Footprint" "azonenberg_pcb:EIA_0603_CAP_NOSILK" (id 2) (at 92.4052 220.98 0)
       (effects (font (size 1.27 1.27)) hide)
     )
@@
       (effects (font (size 1.27 1.27)) (justify left))
     )
-    (property "Footprint" "" (id 2) (at 186.3852 219.71 0)
+    (property "Footprint" "azonenberg_pcb:EIA_0603_CAP_NOSILK" (id 2) (at 186.3852 219.71 0)
       (effects (font (size 1.27 1.27)) hide)
     )
@@
       (effects (font (size 1.524 1.524)))
     )
-    (property "Footprint" "" (id 2) (at 133.35 173.99 0)
+    (property "Footprint" "azonenberg_pcb:BGA_484_22x22_FULLARRAY_1MM" (id 2) (at 133.35 173.99 0)
       (effects (font (size 1.524 1.524)) hide)
     )
@@
       (effects (font (size 1.27 1.27)) (justify left))
     )
-    (property "Footprint" "" (id 2) (at 67.0052 205.74 0)
+    (property "Footprint" "azonenberg_pcb:EIA_1206_CAP_NOSILK" (id 2) (at 67.0052 205.74 0)
       (effects (font (size 1.27 1.27)) hide)
     )
@@
       (effects (font (size 1.27 1.27)) (justify left))
     )
-    (property "Footprint" "" (id 2) (at 186.3852 233.68 0)
+    (property "Footprint" "azonenberg_pcb:EIA_0603_CAP_NOSILK" (id 2) (at 186.3852 233.68 0)
       (effects (font (size 1.27 1.27)) hide)
     )
@@
     (property "Reference" "R46" (id 0) (at 68.58 165.1 90))
     (property "Value" "0" (id 1) (at 73.66 166.37 90))
-    (property "Footprint" "" (id 2) (at 73.66 168.148 90)
+    (property "Footprint" "azonenberg_pcb:EIA_0402_RES_NOSILK" (id 2) (at 73.66 168.148 90)
       (effects (font (size 1.27 1.27)) hide)
     )
@@
       (effects (font (size 1.27 1.27)) (justify left))
     )
-    (property "Footprint" "" (id 2) (at 67.0052 220.98 0)
+    (property "Footprint" "azonenberg_pcb:EIA_0603_CAP_NOSILK" (id 2) (at 67.0052 220.98 0)
       (effects (font (size 1.27 1.27)) hide)
     )
@@
     (property "Reference" "R44" (id 0) (at 68.58 160.02 90))
     (property "Value" "0" (id 1) (at 73.66 161.29 90))
-    (property "Footprint" "" (id 2) (at 73.66 163.068 90)
+    (property "Footprint" "azonenberg_pcb:EIA_0402_RES_NOSILK" (id 2) (at 73.66 163.068 90)
       (effects (font (size 1.27 1.27)) hide)
     )
@@
       (effects (font (size 1.27 1.27)) (justify left))
     )
-    (property "Footprint" "" (id 2) (at 186.3852 205.74 0)
+    (property "Footprint" "azonenberg_pcb:EIA_0603_CAP_NOSILK" (id 2) (at 186.3852 205.74 0)
       (effects (font (size 1.27 1.27)) hide)
     )
@@
       (effects (font (size 1.27 1.27)) (justify left))
     )
-    (property "Footprint" "" (id 2) (at 92.4052 205.74 0)
+    (property "Footprint" "azonenberg_pcb:EIA_0603_CAP_NOSILK" (id 2) (at 92.4052 205.74 0)
       (effects (font (size 1.27 1.27)) hide)
     )
@@
       (effects (font (size 1.27 1.27)) (justify left))
     )
-    (property "Footprint" "" (id 2) (at 298.45 189.23 0)
+    (property "Footprint" "azonenberg_pcb:HEATSINK_WAKEFIELDVETTE_960-23-23-F-AB-0" (id 2) (at 298.45 189.23 0)
       (effects (font (size 1.27 1.27)) hide)
     )
@@
       (effects (font (size 1.27 1.27)) (justify left))
     )
-    (property "Footprint" "" (id 2) (at 172.4152 219.71 0)
+    (property "Footprint" "azonenberg_pcb:EIA_0603_CAP_NOSILK" (id 2) (at 172.4152 219.71 0)
       (effects (font (size 1.27 1.27)) hide)
     )
@@
       (effects (font (size 1.524 1.524)) (justify left))
     )
-    (property "Footprint" "" (id 2) (at 264.16 173.99 0)
+    (property "Footprint" "azonenberg_pcb:BGA_484_22x22_FULLARRAY_1MM" (id 2) (at 264.16 173.99 0)
       (effects (font (size 1.524 1.524)) hide)
     )
@@
       (effects (font (size 1.27 1.27)) (justify left))
     )
-    (property "Footprint" "" (id 2) (at 53.0352 205.74 0)
+    (property "Footprint" "azonenberg_pcb:EIA_1210_CAP_NOSILK" (id 2) (at 53.0352 205.74 0)
       (effects (font (size 1.27 1.27)) hide)
     )
@@
       (effects (font (size 1.524 1.524)) (justify left))
     )
-    (property "Footprint" "" (id 2) (at 82.55 173.99 0)
+    (property "Footprint" "azonenberg_pcb:BGA_484_22x22_FULLARRAY_1MM" (id 2) (at 82.55 173.99 0)
       (effects (font (size 1.524 1.524)) hide)
     )
@@
       (effects (font (size 1.27 1.27)) (justify left))
     )
-    (property "Footprint" "" (id 2) (at 53.0352 220.98 0)
+    (property "Footprint" "azonenberg_pcb:EIA_1210_CAP_NOSILK" (id 2) (at 53.0352 220.98 0)
       (effects (font (size 1.27 1.27)) hide)
     )
@@
       (effects (font (size 1.27 1.27)) (justify left))
     )
-    (property "Footprint" "" (id 2) (at 40.3352 220.98 0)
+    (property "Footprint" "azonenberg_pcb:EIA_1210_CAP_NOSILK" (id 2) (at 40.3352 220.98 0)
       (effects (font (size 1.27 1.27)) hide)
     )
@@
     (property "Reference" "R42" (id 0) (at 58.42 132.08 90))
     (property "Value" "33" (id 1) (at 62.23 133.35 90))
-    (property "Footprint" "" (id 2) (at 62.23 131.572 90)
+    (property "Footprint" "azonenberg_pcb:EIA_0402_RES_NOSILK" (id 2) (at 62.23 131.572 90)
       (effects (font (size 1.27 1.27)) hide)
     )
@@
     (property "Reference" "R39" (id 0) (at 34.29 146.05 90))
     (property "Value" "330" (id 1) (at 34.29 148.59 90))
-    (property "Footprint" "" (id 2) (at 34.29 150.368 90)
+    (property "Footprint" "azonenberg_pcb:EIA_0402_RES_NOSILK" (id 2) (at 34.29 150.368 90)
       (effects (font (size 1.27 1.27)) hide)
     )
@@
     (property "Reference" "R43" (id 0) (at 73.66 140.97 90))
     (property "Value" "33" (id 1) (at 73.66 143.51 90))
-    (property "Footprint" "" (id 2) (at 73.66 145.288 90)
+    (property "Footprint" "azonenberg_pcb:EIA_0402_RES_NOSILK" (id 2) (at 73.66 145.288 90)
       (effects (font (size 1.27 1.27)) hide)
     )
@@
       (effects (font (size 1.524 1.524)))
     )
-    (property "Footprint" "" (id 2) (at 194.31 173.99 0)
+    (property "Footprint" "azonenberg_pcb:BGA_484_22x22_FULLARRAY_1MM" (id 2) (at 194.31 173.99 0)
       (effects (font (size 1.524 1.524)) hide)
     )
@@
       (effects (font (size 1.27 1.27)) (justify left))
     )
-    (property "Footprint" "" (id 2) (at 40.3352 205.74 0)
+    (property "Footprint" "azonenberg_pcb:EIA_1210_CAP_NOSILK" (id 2) (at 40.3352 205.74 0)
       (effects (font (size 1.27 1.27)) hide)
     )
@@
       (effects (font (size 1.27 1.27)) (justify left))
     )
-    (property "Footprint" "" (id 2) (at 40.3352 250.19 0)
+    (property "Footprint" "azonenberg_pcb:EIA_1210_CAP_NOSILK" (id 2) (at 40.3352 250.19 0)
       (effects (font (size 1.27 1.27)) hide)
     )
@@
       (effects (font (size 1.27 1.27)) (justify left))
     )
-    (property "Footprint" "" (id 2) (at 53.0352 234.95 0)
+    (property "Footprint" "azonenberg_pcb:EIA_1206_CAP_NOSILK" (id 2) (at 53.0352 234.95 0)
       (effects (font (size 1.27 1.27)) hide)
     )
@@
       (effects (font (size 1.27 1.27)) (justify left))
     )
-    (property "Footprint" "" (id 2) (at 172.4152 233.68 0)
+    (property "Footprint" "azonenberg_pcb:EIA_0603_CAP_NOSILK" (id 2) (at 172.4152 233.68 0)
       (effects (font (size 1.27 1.27)) hide)
     )
@@
       (effects (font (size 1.27 1.27)) (justify left))
     )
-    (property "Footprint" "" (id 2) (at 79.7052 205.74 0)
+    (property "Footprint" "azonenberg_pcb:EIA_0603_CAP_NOSILK" (id 2) (at 79.7052 205.74 0)
       (effects (font (size 1.27 1.27)) hide)
     )
@@
       (effects (font (size 1.27 1.27)) (justify left))
     )
-    (property "Footprint" "" (id 2) (at 40.3352 234.95 0)
+    (property "Footprint" "azonenberg_pcb:EIA_1206_CAP_NOSILK" (id 2) (at 40.3352 234.95 0)
       (effects (font (size 1.27 1.27)) hide)
     )
@@
     (property "Reference" "R40" (id 0) (at 34.29 151.13 90))
     (property "Value" "4.7K" (id 1) (at 34.29 153.67 90))
-    (property "Footprint" "" (id 2) (at 34.29 155.448 90)
+    (property "Footprint" "azonenberg_pcb:EIA_0402_RES_NOSILK" (id 2) (at 34.29 155.448 90)
       (effects (font (size 1.27 1.27)) hide)
     )
@@
     (property "Reference" "R41" (id 0) (at 34.29 156.21 90))
     (property "Value" "4.7K" (id 1) (at 34.29 158.75 90))
-    (property "Footprint" "" (id 2) (at 34.29 160.528 90)
-      (effects (font (size 1.27 1.27)) hide)
-    )
+    (property "Footprint" "azonenberg_pcb:EIA_0402_RES_NOSILK" (id 2) (at 34.29 160.528 90)
+      (effects (font (size 1.27 1.27)) hide)
+    )
