File: pcb/mainboard/mgmt.kicad_sch (KiCad schematic)
At the start: 75 parts

Commit message: Continued initial work on main board
Parts:
- added C124, C126, C127: 0.47 uF, symbol device:C
- added C125: 4.7 uF, symbol device:C
- added D31, D32, D33, D34: GREEN, symbol device:LED
- added D35, D36, D37, D38: SZESD7471N2T5G, symbol device:D_TVS
- added J48: CONN_01X06, symbol conn:CONN_01X06
- added R124: 1K, symbol device:R
- added R125, R126, R127, R128, R129, R130, R131, R132, R133, R134: 33, symbol device:R
- added R157, R158, R159, R160: 470, symbol device:R
- added U31: ECS-2016MVQ-250-CN, symbol osc-azonenberg:OSC
- added U32: S25FL128SAGBHIA10, symbol memory-azonenberg:S25FLxxxS_BGA24_5x5_VIO
- C100, C102, C103, C104, C105, C106, C107, C108, C109, C82, C83, C87, C88, C89, C91, C92, C94, C95, C96, C99: renamed from C?; footprint azonenberg_pcb:EIA_0402_CAP_NOSILK -> (none)
- C101, C97: renamed from C?; footprint azonenberg_pcb:EIA_1210_CAP_NOSILK -> (none)
- C77, C78, C80, C81, C84, C85, C86: renamed from C?; footprint azonenberg_pcb:EIA_0603_CAP_NOSILK -> (none)
- C79, C93, C98: renamed from C?; footprint azonenberg_pcb:EIA_0805_CAP_NOSILK -> (none)
- C90: renamed from C?; footprint azonenberg_pcb:EIA_1206_CAP_NOSILK -> (none)
- D15, D16, D17, D18: renamed from D?; footprint azonenberg_pcb:EIA_0603_LED -> (none)
- FB6: renamed from FB?; footprint azonenberg_pcb:EIA_0603_INDUCTOR_NOSILK -> (none)
- J10, J8: renamed from J?; footprint azonenberg_pcb:CONN_MOLEX_KK_0470531000 -> (none)
- J11: renamed from J?; footprint azonenberg_pcb:XILINX_JTAG_PTH_MOLEX_0878311420 -> (none)
- J12, J13: renamed from J?; footprint azonenberg_pcb:EIA_0402_JUMPER -> (none)
- J14: renamed from J?; footprint azonenberg_pcb:CONN_RJ45_BELSTEWART_SS-7188S-A-PG4-1-BA-xx -> (none)
- J15: renamed from J?; footprint azonenberg_pcb:CONN_HEADER_2.54MM_2x6_RA_PMOD_HOST -> (none)
- J9: renamed from J?; footprint azonenberg_pcb:CONN_HEADER_2.54MM_1x3 -> (none)
- L3: renamed from L?; footprint azonenberg_pcb:EIA_1210_CAP_NOSILK -> (none)
- R103, R104, R105, R106, R107, R108, R109, R110, R111, R112: renamed from R?; footprint azonenberg_pcb:EIA_0402_RES_NOSILK -> (none)
- R113: renamed from R?; value R -> 33
- TP11, TP12, TP13: renamed from TP?; footprint azonenberg_pcb:CONN_U.FL_TE_1909763-1 -> (none)
- U23: renamed from U?; footprint azonenberg_pcb:BGA_201_10x10_DEPOP_0.65MM_OSHPARK -> (none)
- U24: renamed from U?; footprint azonenberg_pcb:DFN_8_0.5MM_2x3MM_TALL -> (none)
- U25: renamed from U?; footprint azonenberg_pcb:QFN_12_0.5MM_3x3MM -> (none)
- U8: renamed from U?; footprint azonenberg_pcb:BGA_484_22x22_FULLARRAY_1MM -> (none)
Connections:
- net 3V3: now also C124.1, C125.1, C126.1, C127.1, J48.1 (P1), R124.1, U31.1 (E/D#), U31.4 (Vdd), U32.B4 (VDD), U32.E4 (VIO)
- net FAN1_PWM: now also U23.B11 (PC12), D36.2 (A2)
- net FAN1_TACH: now also U8.J21 (IO_L10P_T1_D14_14), D35.2 (A2)
- net FAN2_PWM: now also U23.B7 (PG13), D38.2 (A2)
- net FAN2_TACH: now also U8.J22 (IO_L10N_T1_D15_14), D37.2 (A2)
- net GND: now also C124.2, C125.2, C126.2, C127.2, D31.1 (K), D32.1 (K), D33.1 (K), D34.1 (K), D35.1 (A1), D36.1 (A1), D37.1 (A1), D38.1 (A1), J48.2 (P2), U31.2 (Vss), U32.B3 (VSS)
- net I2C_SCL: now also U23.A2 (PB8)
- net I2C_SDA: now also U23.B3 (PB9)
- net MCU_JTAG_TRST: now also U23.B6 (PB4)
- net MCU_LED0: now also U23.P11 (PF12)
- net MCU_LED1: now also U23.N11 (PF13)
- net MCU_LED2: now also U23.R10 (PF14)
- net MCU_LED3: now also U23.N10 (PF15)
- net MCU_QSPI_CS_N: now also U23.R12 (PE11), U8.R17 (IO_L21P_T3_DQS_14)
- net MCU_QSPI_DQ0: now also U23.R2 (PA2), U8.P19 (IO_L20P_T3_A08_D24_14)
- net MCU_QSPI_DQ1: now also U23.R8 (PB0), U8.R19 (IO_L19N_T3_A09_D25_VREF_14)
- net MCU_QSPI_DQ2: now also U23.M1 (PC2), U8.R18 (IO_L19P_T3_A10_D26_14)
- net MCU_QSPI_DQ3: now also U23.P2 (PA1), U8.L21 (IO_L18N_T2_A11_D27_14)
- net MCU_QSPI_SCK: now also U23.P7 (PB2), U8.P20 (IO_L20N_T3_A07_D23_14)
- net MCU_VDDA: now also U23.M4 (VDDA)
- net FRONTPANEL_CS_N: now reaches U8.E21 (IO_L7P_T1_D09_14)
- net FRONTPANEL_CS_N: now also J48.3 (P3)
- net FRONTPANEL_MOSI: now reaches U8.E22 (IO_L7N_T1_D10_14)
- net FRONTPANEL_MOSI: now also J48.4 (P4)
- net at U8.F19 (IO_L2N_T0_D03_14): now also R133.2
- net FPGA_LED1: now reaches U8.F20 (IO_L4N_T0_D05_14)
- net FPGA_LED1: now also R158.1
- net at U8.G18 (IO_L2P_T0_D02_14): now also R132.2
- net FPGA_LED0: now reaches U8.G20 (IO_L4P_T0_D04_14)
- net FPGA_LED0: now also R157.1
- net FRONTPANEL_SCK: now reaches U8.G22 (IO_L8N_T1_D12_14)
- net FRONTPANEL_SCK: now also J48.6 (P6)
- net at U8.H18 (IO_L1P_T0_D00_MOSI_14): now also R130.2
- net at U8.H19 (IO_L1N_T0_D01_DIN_14): now also R131.2
- net FRONTPANEL_MISO: now reaches U8.H22 (IO_L8P_T1_D11_14)
- net FRONTPANEL_MISO: now also J48.5 (P5)
- net SFP_RX_LOS: now reaches U8.J19 (IO_L3N_T0_DQS_EMCCLK_14)
- net SFP_RX_LOS: now also U23.H3 (PF5)
- net FPGA_LED3: now reaches U8.K19 (IO_L5N_T0_D07_14)
- net FPGA_LED3: now also R160.1
- net FPGA_LED2: now reaches U8.L18 (IO_L5P_T0_D06_14)
- net FPGA_LED2: now also R159.1
- net MCU_IRQ: now reaches U8.M20 (IO_L18P_T2_A12_D28_14)
- net MCU_IRQ: now also U23.P1 (PA0)
- net at U8.M22 (IO_L15N_T2_DQS_DOUT_CSO_B_14): now also R134.2
- net MCU_READY: now reaches U23.B14 (PA8)
- net RX_DAC0_CS_N: now reaches U23.N5 (PA3)
- net DAC_MOSI: now reaches U23.N6 (PA7)
- net RX_DAC1_CS_N: now reaches U23.P5 (PA4)
- net DAC_SCK: now reaches U23.P6 (PA5)
- net DAC_MISO: now reaches U23.R7 (PA6)
- net MCU_CLK_25MHZ: now reaches U23.J1 (PH0)
- net MCU_CLK_25MHZ: now also R125.1
- net SFP_I2C_SCL: now reaches U23.F3 (PF1)
- net SFP_I2C_SDA: now reaches U23.F4 (PF0)
- net SFP_TX_FAULT: now reaches U23.G3 (PF2)
- net FPGA_DONE: now reaches U23.H1 (PF6)
- net SFP_TX_DISABLE: now reaches U23.H2 (PF4)
- net SFP_MOD_ABS: now reaches U23.H4 (PF3)
- net SUPER_SPI_CS_N: now reaches U23.B1 (PE4)
- net TX_DAC_CS_N: now reaches U23.B4 (PE0)
- net SUPER_SPI_SCK: now reaches U23.C3 (PE2)
- net SUPER_SPI_MISO: now reaches U23.D3 (PE5)
- net SUPER_SPI_MOSI: now reaches U23.E3 (PE6)
- new net: D34.2 (A), R160.2
- new net: D32.2 (A), R158.2
- new net: D33.2 (A), R159.2
- new net: D31.2 (A), R157.2
- new net: R124.2, U32.A4 (RESET_N)
- new net: R128.1, U32.C4 (WP_N/DQ2)
- new net: R127.1, U32.D2 (MISO/DQ1)
- new net: R126.1, U32.D3 (MOSI/DQ0)
- new net: R129.1, U32.D4 (RESET_N/DQ3)
- new net: R125.2, U31.3 (CLK)
- new net FLASH_CS_N: R134.1, U32.C2 (CS_N)
- new net FLASH_DQ0: R126.2, R130.1
- new net FLASH_DQ1: R127.2, R131.1
- new net FLASH_DQ2: R128.2, R132.1
- new net FLASH_DQ3: R129.2, R133.1
- new net FLASH_SCK: U32.B2 (SCK)
- no-connect marks 6 -> 116
Other:
- note removed: "TODO: FPGA boot flash (3.3V)"
- moved on the sheet: J15, U23C, U23D, U23G, U23H

Commit message: Calculated power monitor voltage divider
Other:
- company: (none) -> Antikernel Labs
- title: (none) -> Trigger Crossbar
Changed lines of the file:
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@@
 (kicad_sch (version 20211123) (generator eeschema)
   (paper "A3")
+  (title_block
+    (title "Trigger Crossbar")
+    (date "2023-12-17")
+    (rev "0.1")
+    (company "Antikernel Labs")
+    (comment 1 "Andrew D. Zonenberg")
+  )
   (junction (at 106.68 55.88) (diameter 0) (color 0 0 0 0)
   )

Commit message: Fixed typo, changed MCU Vbat to run on 3V3_SB
Connections:
- net 3V3: no longer C82.1, U23.E2 (VBAT)
- new net 3V3_SB: C82.1, U23.E2 (VBAT)
Changed lines of the file:
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@@
   (junction (at 132.08 35.56) (diameter 0) (color 0 0 0 0)
-  )
-  (junction (at 24.13 25.4) (diameter 0) (color 0 0 0 0)
   )
   (junction (at 93.98 147.32) (diameter 0) (color 0 0 0 0)
@@
     (stroke (width 0) (type default) (color 0 0 0 0))
   )
-  (wire (pts (xy 24.13 20.32) (xy 24.13 25.4))
-    (stroke (width 0) (type default) (color 0 0 0 0))
-  )
   (wire (pts (xy 350.52 25.4) (xy 354.33 25.4))
     (stroke (width 0) (type default) (color 0 0 0 0))
@@
     (effects (font (size 1.27 1.27)) (justify right bottom))
   )
-  (label "3V3" (at 29.21 167.64 180)
+  (label "3V3_SB" (at 29.21 167.64 180)
     (effects (font (size 1.27 1.27)) (justify right bottom))
   )
@@
     (effects (font (size 1.27 1.27)) (justify right bottom))
   )
-  (hierarchical_label "3V3" (shape input) (at 24.13 20.32 180)
+  (hierarchical_label "3V3" (shape input) (at 24.13 25.4 180)
     (effects (font (size 1.27 1.27)) (justify right))
   )
@@
     (effects (font (size 1.27 1.27)) (justify right))
   )
+  (hierarchical_label "3V3_SB" (shape input) (at 24.13 20.32 180)
+    (effects (font (size 1.27 1.27)) (justify right))
+  )

Commit message: Began assigning footprints
Parts:
- C100, C102, C103, C104, C105, C106, C107, C108, C109, C124, C126, C127, C82, C83, C87, C88, C89, C91, C92, C94, C95, C96, C99: footprint (none) -> azonenberg_pcb:EIA_0402_CAP_NOSILK
- C101, C97: footprint (none) -> azonenberg_pcb:EIA_1210_CAP_NOSILK
- C125, C77, C78, C81, C84, C86: footprint (none) -> azonenberg_pcb:EIA_0603_CAP_NOSILK
- C79, C80, C85, C90, C93, C98: footprint (none) -> azonenberg_pcb:EIA_0805_CAP_NOSILK
- D15, D16, D17, D18, D31, D32, D33, D34: footprint (none) -> azonenberg_pcb:EIA_0603_LED
- D35, D36, D37, D38: footprint (none) -> azonenberg_pcb:SOD882
- J11: footprint (none) -> azonenberg_pcb:XILINX_JTAG_PTH_MOLEX_0878311420
- J12, J13: footprint (none) -> azonenberg_pcb:EIA_0402_JUMPER
- J14: footprint (none) -> azonenberg_pcb:CONN_RJ45_BELSTEWART_SS-7188S-A-PG4-1-BA-xx
- J15: footprint (none) -> azonenberg_pcb:CONN_HEADER_2.54MM_2x6_RA_PMOD_HOST
- J9: footprint (none) -> azonenberg_pcb:CONN_HEADER_2.54MM_1x3
- R103, R104, R105, R106, R107, R108, R109, R110, R111, R112, R113, R124, R125, R126, R127, R128, R129, R130, R131, R132, R133, R134, R157, R158, R159, R160: footprint (none) -> azonenberg_pcb:EIA_0402_RES_NOSILK
- TP11, TP12, TP13: footprint (none) -> azonenberg_pcb:CONN_U.FL_TE_1909763-1
- U23: footprint (none) -> azonenberg_pcb:BGA_201_10x10_DEPOP_0.65MM_OSHPARK
- U24: footprint (none) -> azonenberg_pcb:DFN_8_0.5MM_2x3MM_TALL
- U25: footprint (none) -> azonenberg_pcb:QFN_12_0.5MM_3x3MM
- U32: footprint (none) -> azonenberg_pcb:BGA_24_6x8_DEPOP1_1MM
- U8: footprint (none) -> azonenberg_pcb:BGA_484_22x22_FULLARRAY_1MM

Commit message: Finished component footprint assignment, started some EM simulations. Ready for schematic review.
Parts:
- FB6: value FERRITE_SMALL2 -> MI0603J601R-10; footprint (none) -> azonenberg_pcb:EIA_0603_INDUCTOR_NOSILK
- J10, J8: footprint (none) -> azonenberg_pcb:CONN_MOLEX_KK_0470531000
- J48: value CONN_01X06 -> CONN_01X10; footprint (none) -> azonenberg_pcb:CONN_MOLEX_PICOBLADE_10POS_0532611071; symbol conn:CONN_01X06 -> conn:CONN_01X10
- L3: footprint (none) -> azonenberg_pcb:EIA_1210_CAP_NOSILK
- U31: value ECS-2016MVQ-250-CN -> ECS-1612MV-250-CN; footprint (none) -> azonenberg_pcb:OSCILLATOR_1.6x1.2
Connections:
- net 3V3: now also J48.2 (P2); no longer J48.1 (P1)
- net 3V3_SB: now also J48.9 (P9)
- net FRONTPANEL_CS_N: now also J48.4 (P4); no longer J48.3 (P3)
- net FRONTPANEL_MISO: now also J48.6 (P6); no longer J48.5 (P5)
- net FRONTPANEL_MOSI: now also J48.5 (P5); no longer J48.4 (P4)
- net FRONTPANEL_SCK: now also J48.7 (P7); no longer J48.6 (P6)
- net GND: now also J48.1 (P1), J48.10 (P10); no longer J48.2 (P2)
- new net SOFT_POWER: J48.3 (P3)
- new net SOFT_RESET: J48.8 (P8)
Changed lines of the file:
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@@
   (title_block
     (title "Trigger Crossbar")
-    (date "2023-12-17")
+    (date "2023-12-18")
     (rev "0.1")
     (company "Antikernel Labs")
@@
     (effects (font (size 1.27 1.27)) (justify right bottom))
   )
-  (label "FRONTPANEL_MOSI" (at 383.54 212.09 180)
+  (label "FRONTPANEL_MOSI" (at 383.54 214.63 180)
     (effects (font (size 1.27 1.27)) (justify right bottom))
   )
@@
     (effects (font (size 1.27 1.27)) (justify right bottom))
   )
-  (label "FRONTPANEL_MISO" (at 383.54 214.63 180)
+  (label "FRONTPANEL_MISO" (at 383.54 217.17 180)
     (effects (font (size 1.27 1.27)) (justify right bottom))
   )
@@
     (effects (font (size 1.27 1.27)) (justify right bottom))
   )
-  (label "FRONTPANEL_CS_N" (at 383.54 209.55 180)
+  (label "FRONTPANEL_CS_N" (at 383.54 212.09 180)
     (effects (font (size 1.27 1.27)) (justify right bottom))
   )
@@
     (effects (font (size 1.27 1.27)) (justify right bottom))
   )
+  (label "GND" (at 383.54 204.47 180)
+    (effects (font (size 1.27 1.27)) (justify right bottom))
+  )
   (label "MCU_QSPI_SCK" (at 354.33 121.92 180)
     (effects (font (size 1.27 1.27)) (justify right bottom))
@@
     (effects (font (size 1.27 1.27)) (justify right bottom))
   )
-  (label "3V3" (at 383.54 204.47 180)
+  (label "3V3" (at 383.54 207.01 180)
     (effects (font (size 1.27 1.27)) (justify right bottom))
   )
@@
     (effects (font (size 1.27 1.27)) (justify right bottom))
   )
-  (label "FRONTPANEL_SCK" (at 383.54 217.17 180)
+  (label "FRONTPANEL_SCK" (at 383.54 219.71 180)
     (effects (font (size 1.27 1.27)) (justify right bottom))
   )
@@
     (effects (font (size 1.27 1.27)) (justify right bottom))
   )
-  (label "GND" (at 383.54 207.01 180)
+  (label "GND" (at 383.54 227.33 180)
     (effects (font (size 1.27 1.27)) (justify right bottom))
   )
@@
     (effects (font (size 1.27 1.27)) (justify right bottom))
   )
+  (label "3V3_SB" (at 383.54 224.79 180)
+    (effects (font (size 1.27 1.27)) (justify right bottom))
+  )
   (label "GND" (at 85.09 262.89 180)
     (effects (font (size 1.27 1.27)) (justify right bottom))
@@
     (effects (font (size 1.27 1.27)) (justify right))
   )
+  (hierarchical_label "SOFT_RESET" (shape output) (at 383.54 222.25 180)
+    (effects (font (size 1.27 1.27)) (justify right))
+  )
+  (hierarchical_label "SOFT_POWER" (shape output) (at 383.54 209.55 180)
+    (effects (font (size 1.27 1.27)) (justify right))
+  )
   (hierarchical_label "GND" (shape input) (at 36.83 254 180)
     (effects (font (size 1.27 1.27)) (justify right))
@@
     (pin "2")
   )
-  (symbol (lib_id "conn:CONN_01X06") (at 388.62 210.82 0) (unit 1)
+  (symbol (lib_id "conn:CONN_01X10") (at 388.62 215.9 0) (unit 1)
     (in_bom yes) (on_board yes) (fields_autoplaced)
-    (property "Reference" "J48" (id 0) (at 390.525 209.9853 0)
+    (property "Reference" "J48" (id 0) (at 390.525 215.0653 0)
       (effects (font (size 1.27 1.27)) (justify left))
     )
-    (property "Value" "CONN_01X06" (id 1) (at 390.525 212.5222 0)
+    (property "Value" "CONN_01X10" (id 1) (at 390.525 217.6022 0)
       (effects (font (size 1.27 1.27)) (justify left))
     )
-    (property "Footprint" "" (id 2) (at 388.62 210.82 0)
+    (property "Footprint" "azonenberg_pcb:CONN_MOLEX_PICOBLADE_10POS_0532611071" (id 2) (at 388.62 215.9 0)
       (effects (font (size 1.27 1.27)) hide)
     )
-    (property "Datasheet" "" (id 3) (at 388.62 210.82 0)
+    (property "Datasheet" "" (id 3) (at 388.62 215.9 0)
       (effects (font (size 1.27 1.27)) hide)
     )
     (pin "1")
+    (pin "10")
     (pin "2")
     (pin "3")
@@
     (pin "5")
     (pin "6")
+    (pin "7")
+    (pin "8")
+    (pin "9")
   )
   (symbol (lib_id "device:C") (at 83.82 95.25 0) (unit 1)
@@
       (effects (font (size 1.27 1.27)) (justify left))
     )
-    (property "Footprint" "" (id 2) (at 69.85 257.81 0)
+    (property "Footprint" "azonenberg_pcb:CONN_MOLEX_KK_0470531000" (id 2) (at 69.85 257.81 0)
       (effects (font (size 1.27 1.27)) hide)
     )
@@
     (in_bom yes) (on_board yes)
     (property "Reference" "FB6" (id 0) (at 34.29 99.6655 0))
-    (property "Value" "FERRITE_SMALL2" (id 1) (at 34.29 106.68 0))
-    (property "Footprint" "" (id 2) (at 34.29 104.14 0)
+    (property "Value" "MI0603J601R-10" (id 1) (at 34.29 106.68 0))
+    (property "Footprint" "azonenberg_pcb:EIA_0603_INDUCTOR_NOSILK" (id 2) (at 34.29 104.14 0)
       (effects (font (size 1.524 1.524)) hide)
     )
@@
       (effects (font (size 1.016 1.016)))
     )
-    (property "Footprint" "" (id 2) (at 69.85 20.32 0)
+    (property "Footprint" "azonenberg_pcb:EIA_1210_CAP_NOSILK" (id 2) (at 69.85 20.32 0)
       (effects (font (size 1.524 1.524)) hide)
     )
@@
       (effects (font (size 1.524 1.524)))
     )
-    (property "Value" "ECS-2016MVQ-250-CN" (id 1) (at 258.445 126.2126 0)
+    (property "Value" "ECS-1612MV-250-CN" (id 1) (at 258.445 126.2126 0)
       (effects (font (size 1.524 1.524)))
     )
-    (property "Footprint" "" (id 2) (at 259.08 130.81 0)
+    (property "Footprint" "azonenberg_pcb:OSCILLATOR_1.6x1.2" (id 2) (at 259.08 130.81 0)
       (effects (font (size 1.524 1.524)) hide)
     )
@@
       (effects (font (size 1.27 1.27)) (justify left))
     )
-    (property "Footprint" "" (id 2) (at 41.91 257.81 0)
+    (property "Footprint" "azonenberg_pcb:CONN_MOLEX_KK_0470531000" (id 2) (at 41.91 257.81 0)
       (effects (font (size 1.27 1.27)) hide)
     )
