File: pcb/mainboard/mgmt.kicad_sch (KiCad schematic)
At the start: 91 parts, among them J10 FAN_01, J11 XILINX_JTAG, J12 JUMPER_0402_SPDT, J13 JUMPER_0402_SPDT, J14 RJ45, J15 PMOD_HOST, J48 CONN_01X10, J8 FAN_01, J9 CONN_01X03, U23 STM32H735-UFBGA176-25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

Commit message: Updated PCB schematic with note about R134 errata
Other:
- note added: "ERRATA: R134 should have connected here"
Changed lines of the file:
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@@
+		)
+	)
+	(text "ERRATA: R134 should have connected here"
+		(exclude_from_sim no)
+		(at 352.806 48.26 0)
+		(effects
+			(font
+				(size 1.27 1.27)
+			)
+			(justify right)
 		)
 	)
