File: pcb/mainboard/psu.kicad_sch (KiCad schematic)
At the start: 83 parts

Commit message: Continued initial work on main board
Parts:
- removed L? (x3): INDUCTOR_PWROUT, symbol passive-azonenberg:INDUCTOR_PWROUT
- added C110: 10 pF C0G, symbol device:C
- added C111, C112: 22 uF, symbol device:C
- added C154, C37: 10 uF, symbol device:C
- added C155: 22 uF 25V, symbol device:C
- added C156, C157: 4.7 uF, symbol device:C
- added D1: GREEN, symbol device:LED
- added D19: CTS520,L3F, symbol device:D_Schottky
- added D2: RED, symbol device:LED
- added FB2, FB4, FB5: FERRITE_SMALL2, symbol passive-azonenberg:FERRITE_SMALL2
- added L4: MLZ2012N4R7LTD25, symbol passive-azonenberg:INDUCTOR_PWROUT
- added R114, R115, R116, R117: R, symbol device:R
- added R118: 20k, symbol device:R
- added R119: 49.9k, symbol device:R
- added R120, R27, R29, R31, R33, R35, R36, R38: 1K, symbol device:R
- added R14, R15: 470, symbol device:R
- added R26: DNP, symbol device:R
- added R28, R30, R32, R34, R37: 10K, symbol device:R
- added R7: 100K, symbol device:R
- added SW1, SW2: SWITCH, symbol passive-azonenberg:SWITCH
- added TP17, TP18, TP19, TP20, TP21, TP22, TP23, TP24, TP8, TP9: U.FL, symbol conn:CONN_COAXIAL
- added U26: LMR70503, symbol power-azonenberg:LMR70503
- added U37: ZLDO1117x50TA, symbol passive-azonenberg:LDO1117-XX
- C1, C16, C17, C18, C2, C22, C23, C24, C3, C4, C5, C6: renamed from C?; footprint azonenberg_pcb:EIA_1812_CAP_NOSILK -> (none)
- C10, C11, C12, C13, C14, C15, C28, C29, C30, C31, C32, C33, C8, C9: renamed from C?; footprint azonenberg_pcb:EIA_1210_CAP_NOSILK -> (none)
- C19, C21, C25, C26, C27: renamed from C?; footprint azonenberg_pcb:EIA_0402_CAP_NOSILK -> (none)
- C20: renamed from C?; footprint azonenberg_pcb:EIA_0603_CAP_NOSILK -> (none)
- C7: renamed from C?; value CP1 -> 25SVPF330M
- FB3: renamed from FB?; footprint azonenberg_pcb:EIA_0603_INDUCTOR_NOSILK -> (none)
- J3: renamed from J?; footprint azonenberg_pcb:CONN_HEADER_2.54MM_1x3 -> (none)
- J4: renamed from J?; footprint azonenberg_pcb:CONN_HEADER_2.54MM_1x5 -> (none)
- R1, R10, R11, R12, R13, R16, R17, R18, R19, R2, R20, R21, R22, R23, R24, R25, R3, R4, R5, R6, R8, R9: renamed from R?; footprint azonenberg_pcb:EIA_0402_RES_NOSILK -> (none)
- TP1, TP2, TP3, TP5, TP6, TP7: renamed from TP?; footprint azonenberg_pcb:TESTPOINT_SMT_0.5MM -> (none)
- U2: renamed from U?; footprint azonenberg_pcb:MODULE_MURATA_MYMGK1R812 -> (none)
- U3, U4, U5, U6, U7: renamed from U?; footprint azonenberg_pcb:MODULE_MURATA_MYMGK00504ERSR -> (none)
- gave numbers to parts that had none: 6
Connections:
- net 12V0: now also C155.1, R114.1, TP17.1 (In), U37.3 (Vin)
- net 12V0_EN: now also U1.10 (PA0), R36.1; no longer U1.6 (PH1)
- net 1V0: now also TP18.1 (In)
- net 1V0_EN: now also U1.20 (PB2), R27.1
- net 1V0_PGOOD: now also U1.39 (PB3), R26.1
- net 1V2_EN: now also U1.19 (PB1), R29.1
- net 1V2_PGOOD: now also U1.40 (PB4), R28.1
- net 1V8: now also TP21.1 (In)
- net 1V8_EN: now also U1.45 (PB8), R31.1
- net 1V8_PGOOD: now also U1.26 (PB13), R30.1
- net 3V3: now also C154.1, C37.1, SW1.2, SW2.2, TP20.1 (In), U26.D2 (VIN)
- net 3V3_EN: now also U1.18 (PB0), R35.1
- net 3V3_PGOOD: now also U1.41 (PB5), R34.1
- net 3V3_SB: now also R26.2, R28.2, R30.2, R32.2, R34.2, R37.2, R7.2, TP8.1 (In)
- net GND: now also C111.2, C112.2, C154.2, C155.2, C156.2, C157.2, C37.2, D1.1 (K), D2.1 (K), L4.2, R115.2, R116.1, R117.1, R120.2, R27.2, R29.2, R31.2, R33.2, R35.2, R36.2, R38.2, TP17.2 (Ext), TP18.2 (Ext), TP19.2 (Ext), TP20.2 (Ext), TP21.2 (Ext), TP22.2 (Ext), TP23.2 (Ext), TP24.2 (Ext), TP8.2 (Ext), TP9.2 (Ext), U26.C1 (GND), U26.C2 (GND), U37.1 (Gnd)
- net GTX_1V0: now also FB5.2, TP23.1 (In)
- net GTX_1V0_EN: now also U1.21 (PB10), R33.1
- net GTX_1V0_PGOOD: now also U1.22 (PB11), R37.1
- net GTX_1V2: now also FB2.2, TP19.1 (In)
- net GTX_1V8: now also FB4.2, TP22.1 (In)
- net GTX_1V8_EN: now also U1.46 (PB9), R38.1
- net GTX_1V8_PGOOD: now also U1.25 (PB12), R32.1
- net SUPER_I2C_SCL: now also U1.30 (PA9)
- net SUPER_I2C_SDA: now also U1.31 (PA10)
- net at R25.1: now also FB5.1
- net at R24.1: now also FB4.1
- net MCU_RST_N: now reaches U1.27 (PB14)
- net at R9.1: now also FB2.1
- net 12V0_VMON: now reaches U1.11 (PA1)
- net 12V0_VMON: now also R114.2, R115.1
- net MCU_READY: now reaches U1.12 (PA2)
- net FPGA_INIT: now reaches U1.13 (PA3)
- net SUPER_SPI_CS_N: now reaches U1.14 (PA4)
- net SUPER_SPI_CS_N: now also R7.1
- net SUPER_SPI_SCK: now reaches U1.15 (PA5)
- net SUPER_SPI_MISO: now reaches U1.16 (PA6)
- net SUPER_SPI_MOSI: now reaches U1.17 (PA7)
- net FPGA_DONE: now reaches U1.29 (PA8)
- net FPGA_RST_N: now reaches U1.32 (PA11)
- net SOFT_RESET: now reaches U1.1 (PC0)
- net SOFT_RESET: now also R116.2, SW1.1
- net SOFT_POWER: now reaches U1.2 (PC13)
- net SOFT_POWER: now also R117.2, SW2.1
- net 3V0_N_EN: now reaches U1.3 (PC14)
- net 3V0_N_EN: now also R120.1, U26.B1 (EN)
- net SUPER_LED0: now reaches U1.5 (PH0)
- net SUPER_LED0: now also R14.2
- new net: C110.1, R118.2, R119.2, U26.A2 (FB)
- new net: D19.1 (K), L4.1, U26.D1 (SW)
- new net: D1.2 (A), R14.1
- new net: D2.2 (A), R15.1
- new net: R118.1, U26.A1 (VREF)
- new net 3V0_N: C110.2, C111.1, C112.1, D19.2 (A), R119.1, TP24.1 (In), U26.B2 (VOUT)
- new net 5V0: C156.1, C157.1, TP9.1 (In), U37.2 (Vout)
- new net SUPER_LED1: R15.2, U1.6 (PH1)
- no-connect marks 0 -> 4
Other:
- note added: "R118 = Rt = 20-100K R119 = Rb = Rt * Vout / Vref Vout = (Rb * 1.19) / Rt so expect -2.96V out"

Commit message: Calculated power monitor voltage divider
Parts:
- R114: value R -> 33K
- R115: value R -> 8.06K
Other:
- company: (none) -> Antikernel Labs
- title: (none) -> Trigger Crossbar
Changed lines of the file:
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@@
 (kicad_sch (version 20211123) (generator eeschema)
   (paper "A2")
+  (title_block
+    (title "Trigger Crossbar")
+    (date "2023-12-17")
+    (rev "0.1")
+    (company "Antikernel Labs")
+    (comment 1 "Andrew D. Zonenberg")
+  )
   (junction (at 187.96 375.92) (diameter 0) (color 0 0 0 0)
   )
@@
       (effects (font (size 1.27 1.27)) (justify left))
     )
-    (property "Value" "R" (id 1) (at 41.148 329.3622 0)
+    (property "Value" "33K" (id 1) (at 41.148 329.3622 0)
       (effects (font (size 1.27 1.27)) (justify left))
     )
@@
       (effects (font (size 1.27 1.27)) (justify left))
     )
-    (property "Value" "R" (id 1) (at 41.148 340.7922 0)
+    (property "Value" "8.06K" (id 1) (at 41.148 340.7922 0)
       (effects (font (size 1.27 1.27)) (justify left))
     )

Commit message: Fixed typo, changed MCU Vbat to run on 3V3_SB
Changed lines of the file:
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@@
+    (stroke (width 0) (type default) (color 0 0 0 0))
+  )
+  (wire (pts (xy 41.91 53.34) (xy 46.99 53.34))
     (stroke (width 0) (type default) (color 0 0 0 0))
   )
@@
     (effects (font (size 1.27 1.27)) (justify right bottom))
   )
-  (label "3V3_SB" (at 41.91 53.34 0)
-    (effects (font (size 1.27 1.27)) (justify left bottom))
-  )
   (label "GND" (at 285.75 204.47 180)
     (effects (font (size 1.27 1.27)) (justify right bottom))
@@
     (effects (font (size 1.27 1.27)) (justify right))
   )
+  (hierarchical_label "3V3_SB" (shape output) (at 46.99 53.34 0)
+    (effects (font (size 1.27 1.27)) (justify left))
+  )
   (hierarchical_label "FPGA_RST_N" (shape output) (at 35.56 378.46 180)

Commit message: Began assigning footprints
Parts:
- C1, C155, C16, C17, C18, C2, C22, C23, C24, C3, C4, C5, C6: footprint (none) -> azonenberg_pcb:EIA_1812_CAP_NOSILK
- C10, C11, C12, C13, C14, C15, C28, C29, C30, C31, C32, C33, C8, C9: footprint (none) -> azonenberg_pcb:EIA_1210_CAP_NOSILK
- C110, C19, C21, C25, C26, C27: footprint (none) -> azonenberg_pcb:EIA_0402_CAP_NOSILK
- C111, C112, C154, C37: footprint (none) -> azonenberg_pcb:EIA_0805_CAP_NOSILK
- C156, C157, C20: footprint (none) -> azonenberg_pcb:EIA_0603_CAP_NOSILK
- C7: footprint (none) -> azonenberg_pcb:CAP_AL_10MM_SMT
- D1, D2: footprint (none) -> azonenberg_pcb:EIA_0603_LED
- D19: footprint (none) -> azonenberg_pcb:SOD882
- FB3: footprint (none) -> azonenberg_pcb:EIA_0603_INDUCTOR_NOSILK
- J1: footprint (none) -> azonenberg_pcb:CONN_MOLEX_MINIFITJR_8POS_0039291087
- J2: footprint (none) -> azonenberg_pcb:CONN_MOLEX_PICOBLADE_5POS_0532610571
- J3, TP4: footprint (none) -> azonenberg_pcb:CONN_HEADER_2.54MM_1x3
- J4: footprint (none) -> azonenberg_pcb:CONN_HEADER_2.54MM_1x5
- R1, R10, R11, R114, R115, R118, R119, R12, R120, R13, R14, R15, R16, R17, R18, R19, R2, R20, R21, R22, R23, R24, R25, R26, R27, R28, R29, R3, R30, R31, R32, R33, R34, R35, R36, R37, R38, R4, R5, R6, R7, R8, R9: footprint (none) -> azonenberg_pcb:EIA_0402_RES_NOSILK
- R116, R117: value R -> 10K; footprint (none) -> azonenberg_pcb:EIA_0402_RES_NOSILK
- TP1, TP2, TP3, TP5, TP6, TP7: footprint (none) -> azonenberg_pcb:TESTPOINT_SMT_0.5MM
- TP17, TP18, TP19, TP20, TP21, TP22, TP23, TP24, TP8, TP9: footprint (none) -> azonenberg_pcb:CONN_U.FL_TE_1909763-1
- U1: footprint (none) -> azonenberg_pcb:QFN_48_0.5MM_7x7MM
- U2: footprint (none) -> azonenberg_pcb:MODULE_MURATA_MYMGK1R812
- U26: footprint (none) -> azonenberg_pcb:BGA_8_1.65x0.865_0.4MM_TI_YFX
- U3, U4, U5, U6, U7: footprint (none) -> azonenberg_pcb:MODULE_MURATA_MYMGK00504ERSR
- U37: footprint (none) -> azonenberg_pcb:SOT223-4

Commit message: Finished component footprint assignment, started some EM simulations. Ready for schematic review.
Parts:
- F1: footprint (none) -> azonenberg_pcb:EIA_0603_CAP_NOSILK
- FB1, FB2, FB4, FB5: value FERRITE_SMALL2 -> BLM31KN271SH1L; footprint (none) -> azonenberg_pcb:EIA_1206_CAP_NOSILK
- L4: footprint (none) -> azonenberg_pcb:EIA_0805_INDUCTOR_NOSILK
- SW1, SW2: footprint (none) -> azonenberg_pcb:SWITCH_RAFI_MICON_5
Changed lines of the file:
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@@
   (title_block
     (title "Trigger Crossbar")
-    (date "2023-12-17")
+    (date "2023-12-18")
     (rev "0.1")
     (company "Antikernel Labs")
@@
     (effects (font (size 1.27 1.27)) (justify left bottom))
   )
-  (label "SOFT_RESET" (at 109.22 322.58 0)
-    (effects (font (size 1.27 1.27)) (justify left bottom))
-  )
   (label "SUPER_UART_RX" (at 78.74 368.3 180)
     (effects (font (size 1.27 1.27)) (justify right bottom))
@@
     (effects (font (size 1.27 1.27)) (justify right bottom))
   )
-  (label "SOFT_POWER" (at 130.81 322.58 0)
-    (effects (font (size 1.27 1.27)) (justify left bottom))
-  )
   (label "GND" (at 130.81 331.47 0)
     (effects (font (size 1.27 1.27)) (justify left bottom))
@@
     (effects (font (size 1.27 1.27)) (justify right))
   )
+  (hierarchical_label "SOFT_POWER" (shape input) (at 130.81 322.58 0)
+    (effects (font (size 1.27 1.27)) (justify left))
+  )
+  (hierarchical_label "SOFT_RESET" (shape input) (at 109.22 322.58 0)
+    (effects (font (size 1.27 1.27)) (justify left))
+  )
   (hierarchical_label "GTX_1V0" (shape output) (at 327.66 196.85 0)
     (effects (font (size 1.27 1.27)) (justify left))
@@
     (in_bom yes) (on_board yes)
     (property "Reference" "FB1" (id 0) (at 72.39 19.9222 0))
-    (property "Value" "FERRITE_SMALL2" (id 1) (at 71.12 26.67 0))
-    (property "Footprint" "" (id 2) (at 72.39 24.13 0)
+    (property "Value" "BLM31KN271SH1L" (id 1) (at 71.12 26.67 0))
+    (property "Footprint" "azonenberg_pcb:EIA_1206_CAP_NOSILK" (id 2) (at 72.39 24.13 0)
       (effects (font (size 1.524 1.524)) hide)
     )
@@
     (property "Reference" "SW1" (id 0) (at 101.761 318.135 0))
     (property "Value" "SWITCH" (id 1) (at 104.2979 318.135 0))
-    (property "Footprint" "" (id 2) (at 106.68 318.77 0)
+    (property "Footprint" "azonenberg_pcb:SWITCH_RAFI_MICON_5" (id 2) (at 106.68 318.77 0)
       (effects (font (size 1.27 1.27)) hide)
     )
@@
       (effects (font (size 1.016 1.016)))
     )
-    (property "Footprint" "" (id 2) (at 290.83 274.32 0)
+    (property "Footprint" "azonenberg_pcb:EIA_0805_INDUCTOR_NOSILK" (id 2) (at 290.83 274.32 0)
       (effects (font (size 1.524 1.524)) hide)
     )
@@
     (property "Reference" "F1" (id 0) (at 58.42 19.9222 0))
     (property "Value" "2A" (id 1) (at 58.42 22.4591 0))
-    (property "Footprint" "" (id 2) (at 60.325 24.13 0)
+    (property "Footprint" "azonenberg_pcb:EIA_0603_CAP_NOSILK" (id 2) (at 60.325 24.13 0)
       (effects (font (size 1.524 1.524)) hide)
     )
@@
     (in_bom yes) (on_board yes)
     (property "Reference" "FB5" (id 0) (at 322.58 192.6422 0))
-    (property "Value" "FERRITE_SMALL2" (id 1) (at 321.31 199.39 0))
-    (property "Footprint" "" (id 2) (at 322.58 196.85 0)
+    (property "Value" "BLM31KN271SH1L" (id 1) (at 321.31 199.39 0))
+    (property "Footprint" "azonenberg_pcb:EIA_1206_CAP_NOSILK" (id 2) (at 322.58 196.85 0)
       (effects (font (size 1.524 1.524)) hide)
     )
@@
     (in_bom yes) (on_board yes)
     (property "Reference" "FB4" (id 0) (at 322.58 130.4122 0))
-    (property "Value" "FERRITE_SMALL2" (id 1) (at 321.31 137.16 0))
-    (property "Footprint" "" (id 2) (at 322.58 134.62 0)
+    (property "Value" "BLM31KN271SH1L" (id 1) (at 321.31 137.16 0))
+    (property "Footprint" "azonenberg_pcb:EIA_1206_CAP_NOSILK" (id 2) (at 322.58 134.62 0)
       (effects (font (size 1.524 1.524)) hide)
     )
@@
     (in_bom yes) (on_board yes)
     (property "Reference" "FB2" (id 0) (at 139.7 159.6222 0))
-    (property "Value" "FERRITE_SMALL2" (id 1) (at 138.43 166.37 0))
-    (property "Footprint" "" (id 2) (at 139.7 163.83 0)
+    (property "Value" "BLM31KN271SH1L" (id 1) (at 138.43 166.37 0))
+    (property "Footprint" "azonenberg_pcb:EIA_1206_CAP_NOSILK" (id 2) (at 139.7 163.83 0)
       (effects (font (size 1.524 1.524)) hide)
     )
@@
     (property "Reference" "SW2" (id 0) (at 123.351 318.135 0))
     (property "Value" "SWITCH" (id 1) (at 125.8879 318.135 0))
-    (property "Footprint" "" (id 2) (at 128.27 318.77 0)
+    (property "Footprint" "azonenberg_pcb:SWITCH_RAFI_MICON_5" (id 2) (at 128.27 318.77 0)
       (effects (font (size 1.27 1.27)) hide)
     )
