File: pcb/mainboard/mainboard.kicad_sch (KiCad schematic)
At the start: 10 parts, among them M2 LOGO, M3 LOGO, M4 LOGO, M5 LOGO

Commit message: Continued layout review, various routing and silkscreen cleanup. DRC clean.
Parts:
- added M10, M11, M6, M7, M8, M9: FIDUCIAL, azonenberg_pcb:FIDUCIAL_1MM, symbol special-azonenberg:MECHANICAL
Changed lines of the file:
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@@
+    )
+  )
+  (symbol (lib_id "special-azonenberg:MECHANICAL") (at 172.72 125.73 0) (unit 1)
+    (in_bom yes) (on_board yes) (fields_autoplaced)
+    (property "Reference" "M9" (id 0) (at 175.895 124.8953 0)
+      (effects (font (size 1.27 1.27)) (justify left))
+    )
+    (property "Value" "FIDUCIAL" (id 1) (at 175.895 127.4322 0)
+      (effects (font (size 1.27 1.27)) (justify left))
+    )
+    (property "Footprint" "azonenberg_pcb:FIDUCIAL_1MM" (id 2) (at 172.72 125.73 0)
+      (effects (font (size 1.27 1.27)) hide)
+    )
+    (property "Datasheet" "" (id 3) (at 172.72 125.73 0)
+      (effects (font (size 1.27 1.27)) hide)
     )
   )
@@
     (pin "1")
   )
+  (symbol (lib_id "special-azonenberg:MECHANICAL") (at 156.21 125.73 0) (unit 1)
+    (in_bom yes) (on_board yes) (fields_autoplaced)
+    (property "Reference" "M6" (id 0) (at 159.385 124.8953 0)
+      (effects (font (size 1.27 1.27)) (justify left))
+    )
+    (property "Value" "FIDUCIAL" (id 1) (at 159.385 127.4322 0)
+      (effects (font (size 1.27 1.27)) (justify left))
+    )
+    (property "Footprint" "azonenberg_pcb:FIDUCIAL_1MM" (id 2) (at 156.21 125.73 0)
+      (effects (font (size 1.27 1.27)) hide)
+    )
+    (property "Datasheet" "" (id 3) (at 156.21 125.73 0)
+      (effects (font (size 1.27 1.27)) hide)
+    )
+  )
+  (symbol (lib_id "special-azonenberg:MECHANICAL") (at 156.21 142.24 0) (unit 1)
+    (in_bom yes) (on_board yes) (fields_autoplaced)
+    (property "Reference" "M8" (id 0) (at 159.385 141.4053 0)
+      (effects (font (size 1.27 1.27)) (justify left))
+    )
+    (property "Value" "FIDUCIAL" (id 1) (at 159.385 143.9422 0)
+      (effects (font (size 1.27 1.27)) (justify left))
+    )
+    (property "Footprint" "azonenberg_pcb:FIDUCIAL_1MM" (id 2) (at 156.21 142.24 0)
+      (effects (font (size 1.27 1.27)) hide)
+    )
+    (property "Datasheet" "" (id 3) (at 156.21 142.24 0)
+      (effects (font (size 1.27 1.27)) hide)
+    )
+  )
+  (symbol (lib_id "special-azonenberg:MECHANICAL") (at 156.21 133.35 0) (unit 1)
+    (in_bom yes) (on_board yes) (fields_autoplaced)
+    (property "Reference" "M7" (id 0) (at 159.385 132.5153 0)
+      (effects (font (size 1.27 1.27)) (justify left))
+    )
+    (property "Value" "FIDUCIAL" (id 1) (at 159.385 135.0522 0)
+      (effects (font (size 1.27 1.27)) (justify left))
+    )
+    (property "Footprint" "azonenberg_pcb:FIDUCIAL_1MM" (id 2) (at 156.21 133.35 0)
+      (effects (font (size 1.27 1.27)) hide)
+    )
+    (property "Datasheet" "" (id 3) (at 156.21 133.35 0)
+      (effects (font (size 1.27 1.27)) hide)
+    )
+  )
   (symbol (lib_id "conn:CONN_01X01") (at 227.33 132.08 0) (unit 1)
     (in_bom yes) (on_board yes) (fields_autoplaced)
@@
     )
     (pin "1")
+  )
+  (symbol (lib_id "special-azonenberg:MECHANICAL") (at 172.72 133.35 0) (unit 1)
+    (in_bom yes) (on_board yes) (fields_autoplaced)
+    (property "Reference" "M10" (id 0) (at 175.895 132.5153 0)
+      (effects (font (size 1.27 1.27)) (justify left))
+    )
+    (property "Value" "FIDUCIAL" (id 1) (at 175.895 135.0522 0)
+      (effects (font (size 1.27 1.27)) (justify left))
+    )
+    (property "Footprint" "azonenberg_pcb:FIDUCIAL_1MM" (id 2) (at 172.72 133.35 0)
+      (effects (font (size 1.27 1.27)) hide)
+    )
+    (property "Datasheet" "" (id 3) (at 172.72 133.35 0)
+      (effects (font (size 1.27 1.27)) hide)
+    )
+  )
+  (symbol (lib_id "special-azonenberg:MECHANICAL") (at 172.72 142.24 0) (unit 1)
+    (in_bom yes) (on_board yes) (fields_autoplaced)
+    (property "Reference" "M11" (id 0) (at 175.895 141.4053 0)
+      (effects (font (size 1.27 1.27)) (justify left))
+    )
+    (property "Value" "FIDUCIAL" (id 1) (at 175.895 143.9422 0)
+      (effects (font (size 1.27 1.27)) (justify left))
+    )
+    (property "Footprint" "azonenberg_pcb:FIDUCIAL_1MM" (id 2) (at 172.72 142.24 0)
+      (effects (font (size 1.27 1.27)) hide)
+    )
+    (property "Datasheet" "" (id 3) (at 172.72 142.24 0)
+      (effects (font (size 1.27 1.27)) hide)
+    )
   )
   (symbol (lib_id "special-azonenberg:MECHANICAL") (at 196.85 142.24 0) (unit 1)
@@
       (reference "M5") (unit 1) (value "LOGO") (footprint "w_logo:Logo_silk_WEEE_3.4x5mm")
     )
+    (path "/6eee91e2-e2dd-437a-af95-33d43a6816ac"
+      (reference "M6") (unit 1) (value "FIDUCIAL") (footprint "azonenberg_pcb:FIDUCIAL_1MM")
+    )
+    (path "/882ff0bb-2159-4e4e-b9bc-a7703b5ac128"
+      (reference "M7") (unit 1) (value "FIDUCIAL") (footprint "azonenberg_pcb:FIDUCIAL_1MM")
+    )
+    (path "/77b51363-05a7-4c0b-903a-b2768b5a8a6e"
+      (reference "M8") (unit 1) (value "FIDUCIAL") (footprint "azonenberg_pcb:FIDUCIAL_1MM")
+    )
+    (path "/2aec54e3-71b1-44bd-ab9a-db9d450ee311"
+      (reference "M9") (unit 1) (value "FIDUCIAL") (footprint "azonenberg_pcb:FIDUCIAL_1MM")
+    )
+    (path "/9427dafa-7565-4829-be67-0688d05ebc06"
+      (reference "M10") (unit 1) (value "FIDUCIAL") (footprint "azonenberg_pcb:FIDUCIAL_1MM")
+    )
+    (path "/e11141d8-229b-4ca1-bcf0-967fe3188fa1"
+      (reference "M11") (unit 1) (value "FIDUCIAL") (footprint "azonenberg_pcb:FIDUCIAL_1MM")
+    )
     (path "/eb063380-1a9b-4dc0-8558-af6481d57a5e"
